File: esquematico.brd (EAGLE design)
At the start: 100 x 80 mm, 11 parts

Commit message: listo el pcb para el plano de tierra
Parts:
- removed U$3: BNCPTH, SparkFun-Connectors:BNC
- added BNC_TRANSDUCER: BNCPTH, SparkFun-Connectors:BNC
- R3: value (none) -> 127
- moved TRANSDUCER 210.7 mm to (92.7, 20.3), turned to 90 degrees
- moved PW_SW 188.2 mm to (92.7, 5.08), turned to 90 degrees
- moved SELECTOR 146.0 mm to (63.5, 6.35)
- moved R2 136.0 mm to (66.0, 17.8)
- moved GENERATOR 115.2 mm to (91.4, 31.8)
- moved R1 115.1 mm to (45.7, 17.8)
- moved VAR_RES 115.0 mm to (6.35, 12.7), turned to 270 degrees
- moved R3 99.2 mm to (26.7, 17.8)
- moved OUT_OSC 83.6 mm to (12.7, 31.8)
- moved COUNTER 76.4 mm to (35.6, 31.8)
Connections:
- net N$1: now also BNC_TRANSDUCER.GND; no longer U$3.GND
- net N$7: now also BNC_TRANSDUCER.S; no longer U$3.S
Other:
- board size 100 x 80 mm -> 100 x 43.2 mm

Commit message: anade el plano de tierra
Routing:
- added copper zone on layer 16, net GND
Changed lines of the file:
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@@
 <contactref element="GENERATOR" pad="S"/>
 <contactref element="PW_SW" pad="2"/>
-<wire x1="91.44" y1="31.75" x2="93.98" y2="7.58" width="0" layer="19" extent="1-1"/>
+<wire x1="93.98" y1="7.58" x2="91.44" y2="31.75" width="0" layer="19" extent="1-1"/>
 </signal>
 <signal name="N$3">
@@
 <contactref element="VAR_RES" pad="1"/>
 <contactref element="SELECTOR" pad="1"/>
-<wire x1="58.5" y1="5.06" x2="5.08" y2="15.2" width="0" layer="19" extent="1-1"/>
+<wire x1="5.08" y1="15.2" x2="58.5" y2="5.06" width="0" layer="19" extent="1-1"/>
 </signal>
 <signal name="N$9">
@@
 <contactref element="OUT_OSC" pad="GND"/>
 <contactref element="R3" pad="P$1"/>
-<wire x1="71.12" y1="17.78" x2="21.59" y2="17.78" width="0" layer="19" extent="1-1"/>
-<wire x1="10.16" y1="31.75" x2="71.12" y2="17.78" width="0" layer="19" extent="1-1"/>
-<wire x1="33.02" y1="31.75" x2="71.12" y2="17.78" width="0" layer="19" extent="1-1"/>
-<wire x1="88.9" y1="31.75" x2="33.02" y2="31.75" width="0" layer="19" extent="1-1"/>
+<polygon width="0.4064" layer="16">
+<vertex x="-5.08" y="44.45"/>
+<vertex x="-6.35" y="44.45"/>
+<vertex x="-6.35" y="-3.81"/>
+<vertex x="104.14" y="-3.81"/>
+<vertex x="105.41" y="-3.81"/>
+<vertex x="105.41" y="45.72"/>
+<vertex x="-5.08" y="45.72"/>
+</polygon>
 </signal>
 <signal name="N$1">
@@
 <contactref element="R2" pad="P$1"/>
 <contactref element="VAR_RES" pad="2"/>
-<wire x1="5.08" y1="10.2" x2="93.98" y2="17.82" width="0" layer="19" extent="1-1"/>
-<wire x1="60.96" y1="17.78" x2="5.08" y2="10.2" width="0" layer="19" extent="1-1"/>
+<wire x1="60.96" y1="17.78" x2="93.98" y2="17.82" width="0" layer="19" extent="1-1"/>
 <wire x1="50.8" y1="17.78" x2="60.96" y2="17.78" width="0" layer="19" extent="1-1"/>
-<wire x1="60.96" y1="31.75" x2="50.8" y2="17.78" width="0" layer="19" extent="1-1"/>
+<wire x1="60.96" y1="31.75" x2="60.96" y2="17.78" width="0" layer="19" extent="1-1"/>
+<wire x1="5.08" y1="10.2" x2="50.8" y2="17.78" width="0" layer="19" extent="1-1"/>
 </signal>
 </signals>

Commit message: el proyecto se termina la revision 1.0
Parts:
- moved VAR_RES 0.64 mm to (6.99, 12.7)
Routing:
- net N$9: track 0.00 -> 115.8 mm
- net N$1: track 0.00 -> 111.8 mm
- net N$3: track 0.00 -> 107.2 mm
- net N$7: track 0.00 -> 74.2 mm
- net N$8: track 0.00 -> 68.0 mm
- net N$2: track 0.00 -> 28.6 mm
